File: Kicad/CH376S ISA.kicad_pcb (KiCad board)
At the start: 2 copper layers, 29 parts, among them J1 Bus_ISA_8bit, J2 ROM CS, J3 Conn_02x04_Odd_Even, U1 CH376, U13 74LS138, U14 74LS138, U15 74LS138, U2 LM1117-3.3, U3 74LS139, U4 74LS138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

Commit message: first draft done
Parts:
- removed C3: 0.1uF, Capacitor_THT:C_Disc_D4.3mm_W1.9mm_P5.00mm
- removed J3: Conn_02x04_Odd_Even, Connector_PinHeader_2.54mm:PinHeader_2x04_P2.54mm_Vertical
- removed U6: 28C64, Package_DIP:DIP-28_W15.24mm
- added R: L, Motherboard:Large_Via, F.Cu at (197.9, 85.1)
- added R: L, Motherboard:Large_Via, F.Cu at (197.9, 142.2)
- U3: value 74LS139 -> 28C256; footprint Package_DIP:DIP-16_W7.62mm -> Package_DIP:DIP-28_W15.24mm
- moved C16 77.5 mm to (188.7, 83.9), turned to 270 degrees
- moved C10 72.4 mm to (134.7, 116.1)
- moved C8 59.6 mm to (144.9, 116.1)
- moved U5 54.9 mm to (185.4, 81.3), turned to 270 degrees
- moved U4 49.9 mm to (142.2, 119.4)
- moved J2 49.8 mm to (185.4, 92.2), turned to 270 degrees
- moved C9 49.3 mm to (114.4, 116.1)
- moved U3 25.9 mm to (137.2, 83.8), turned to 270 degrees
- moved C14 19.9 mm to (140.5, 94.1), turned to 270 degrees
- moved C15 14.4 mm to (124.5, 116.1)
- moved U13 10.2 mm to (132.1, 119.4)
- moved U14 10.2 mm to (121.9, 119.4)
- moved U15 10.2 mm to (111.8, 119.4)
- moved J1 0.80 mm to (177.8, 146.1)
Connections:
- J1 pad 42: Net-(J1-Pad42) -> /AEN
- U13 pad 5: /GND -> /AEN
- U15 pad 7: /IO_00EX -> /CH376CS
- U3 pad 1: /IO_00EX -> /GND
- U3 pad 10: (no net) -> /A0
- U3 pad 11: (no net) -> /D0
- U3 pad 12: (no net) -> /D1
- U3 pad 13: (no net) -> /D2
- U3 pad 14: (no net) -> /GND
- U3 pad 15: (no net) -> /D3
- U3 pad 16: /5+ -> /D4
- U3 pad 2: /A0 -> /A12
- U3 pad 3: /A1 -> /A7
- U3 pad 4: /E0 -> /A6
- U3 pad 5: /E1 -> /A5
- U3 pad 6: /E2 -> /A4
- U3 pad 7: /E3 -> /A3
- U3 pad 8: /GND -> /A2
- U3 pad 9: (no net) -> /A1
- U4 pad 5: /GND -> /AEN
Routing:
- net /GND: track 185.7 -> 399.1 mm, vias 8 -> 17
- net /A2: track 0.76 -> 156.3 mm, vias 0 -> 6
- net /5+: track 166.4 -> 313.2 mm, vias 6 -> 12
- net /D2: track 7.86 -> 129.5 mm, vias 1 -> 6
- net /A13: track 0.72 -> 122.1 mm, vias 0 -> 6
- net /A14: track 0.72 -> 119.6 mm, vias 0 -> 4
- net /D1: track 8.62 -> 125.2 mm, vias 1 -> 6
- net /A15: track 0.72 -> 117.2 mm, vias 0 -> 4
- net /D7: track 4.05 -> 115.8 mm, vias 1 -> 6
- net /D5: track 5.57 -> 117.4 mm, vias 1 -> 6
- net /D3: track 7.10 -> 118.9 mm, vias 1 -> 6
- net /D6: track 4.81 -> 116.6 mm, vias 1 -> 6
- net /D4: track 6.34 -> 118.1 mm, vias 1 -> 6
- net /D0: track 9.64 -> 120.9 mm, vias 1 -> 4
- net /ROM_CS_0XEX: track 0.00 -> 88.6 mm, vias 0 -> 3
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Other:
- board outline added: 104 x 73.9 mm
- board text added: "0XE0..."
- board text added: "0XE2..."
- board text added: "0XE4..."
- board text added: "0XE6..."
- board text added: "0XE8..."
- board text added: "0XEA..."
- board text added: "0XEC..."
- board text added: "0XEE..."
- board text added: "8K ROM"
- board text added: "EMM COMPUTERS CH376 ISA Module Copyright (C) 2023 EMM www.homebrew8088.com"
- board text removed: "E0"
- board text removed: "E1"
- board text removed: "E2"
- board text removed: "E3"
- board text removed: "EMM COMPUTERS CH376 Module Copyright (C) 2023 EMM www.homebrew8088.com"
